File: keyboard/dulcimer/circuit/dulcimer.kicad_pcb (KiCad board)
At the start: 2 copper layers, 146 x 50.8 mm, 24 parts, among them IC1 MEGA32-P, X1 12MHz

Commit message: Corrected the orientation of the LED connector
Fixes after first prototypes where built:
 The LED connector was wrongly rotated by 180°. This is corrected now.
 Added drawing on how to mount the compontents to the PCB
Parts:
- JP6: value JUMPER -> Reset
- JP7: value CONN_02X03 -> ISP
- JP8: value CONN_01X02 -> 6.3mm
- moved JP3 7.63 mm to (191.8, 58.4), turned to 90 degrees
Routing:
- net VCC: track 243.8 -> 229.4 mm
- net Net-(JP3-Pad3): track 43.8 -> 37.4 mm
- net Net-(JP3-Pad4): track 47.1 -> 41.0 mm
- net Net-(JP3-Pad1): track 36.9 -> 31.2 mm
Other:
- board text added: "20191229"
- board text added: "Rev 3"
- board text added: "by R. Schaten & nuess0r"
- board text removed: "20161202"
- board text removed: "Rev 2"
- board text removed: "by Ronald Schaten"
